File: Platine.kicad_pcb (KiCad board)
At the start: 4 copper layers, 299.9 x 215.6 mm, 190 parts, among them J1 GND +12V, J10 RJ45_LED_Shielded, J11 Serial 5, J12 Serial 6, J13 Serial 7, J14 Serial 8, J15 CAN 1, J16 Conn_01x02, J17 Conn_01x02, J18 Conn_01x02, J19 Conn_01x02, J2 Conn_01x09, J20 Conn_01x02, J21 Conn_01x02, J22 Conn_01x02, J23 Conn_01x02, J24 Conn_01x02, J25 Conn_01x02, J26 Conn_01x02, J27 Conn_01x02, J28 Conn_01x02, J29 Conn_01x02, J3 Display128x64_I2C, J30 Conn_01x02, J31 Conn_01x02, J32 +12V, J33 GND, J34 Conn_01x02, J35 Conn_01x02, J36 Conn_01x02, J37 Conn_01x02, J38 Conn_01x02, J39 Conn_01x02, J4 +5V, J40 Conn_01x02, J41 Conn_01x02, J42 Conn_01x02, J43 Conn_01x02, J44 Conn_01x02, J45 Conn_01x02, J46 Conn_01x02, J47 Conn_01x02, J48 Conn_01x02, J49 Conn_01x02, J5 Serial 2, J50 Conn_01x02, J51 Conn_01x02, J52 Conn_01x02, J53 Conn_01x02, J54 Conn_01x02, J55 Conn_01x02, J56 Conn_01x02, J57 Conn_01x02, J58 +12V, J59 GND, J6 Serial 3, J60 Conn_01x02, J61 Conn_01x02, J62 Conn_01x02, J63 Conn_01x02, J64 Conn_01x02, J65 Conn_01x02, J66 Conn_01x02, J67 Conn_01x02, J68 Relais 1, J69 Relais 2, J7 Conn_01x24_Female, J70 Relais 3, J71 Relais 4, J72 Relais 5, J73 Relais 6, J74 Relais 7, J75 Relais 8, J76 +3.3V, J77 GND, J78 +3.3V, J79 GND, J8 Conn_01x24_Female, J80 +5V, J81 GND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

Commit message: ..
Parts:
- removed C10, C11, C12: C_Polarized, Capacitor_THT:CP_Radial_D6.3mm_P2.50mm
- removed C7, C8: 100nF, Capacitor_SMD:C_0805_2012Metric_Pad1.18x1.45mm_HandSolder
- removed D42, D43, D44: LED, LED_THT:LED_D3.0mm
- removed F1: 12V, Fuse:Fuseholder_TR5_Littelfuse_No560_No460
- removed F2: 5V, Fuse:Fuseholder_TR5_Littelfuse_No560_No460
- removed F3: 3.3V, Fuse:Fuseholder_TR5_Littelfuse_No560_No460
- removed J74: Relais 7, AA_EigeneBauteile:TerminalBlock_MetzConnect_Type166_1x03_P3.50mm_Horizontal
- removed J75: Relais 8, AA_EigeneBauteile:TerminalBlock_MetzConnect_Type166_1x03_P3.50mm_Horizontal
- removed J76: +3.3V, AA_EigeneBauteile:TerminalBlock_MetzConnect_Type166_1x03_P3.50mm_Horizontal
- removed J77, J93, J95: GND, AA_EigeneBauteile:TerminalBlock_MetzConnect_Type166_1x03_P3.50mm_Horizontal
- removed J78: +3.3V, AA_EigeneBauteile:TerminalBlock_MetzConnect_Type166x1x05_P3.50mm_Horizontal
- removed J79, J81, J90: GND, AA_EigeneBauteile:TerminalBlock_MetzConnect_Type166x1x05_P3.50mm_Horizontal
- removed J80: +5V, AA_EigeneBauteile:TerminalBlock_MetzConnect_Type166x1x05_P3.50mm_Horizontal
- removed J82: CAN-Module1, AA_EigeneBauteile:CAN_Pinsocket_SMD
- removed J83: CAN-Module2, AA_EigeneBauteile:CAN_Pinsocket_SMD
- removed J84: CAN 2, TerminalBlock_MetzConnect:TerminalBlock_MetzConnect_Type059_RT06306HBWC_1x06_P3.50mm_Horizontal
- removed J85: 1Wire, AA_EigeneBauteile:TerminalBlock_MetzConnect_Type166_1x03_P3.50mm_Horizontal
- removed J86: SPI, AA_EigeneBauteile:SPI_Pinsocket_SMD
- removed J87, J88, J97: Conn_01x02, Connector_PinHeader_2.54mm:PinHeader_1x02_P2.54mm_Vertical
- removed J89: +12V, AA_EigeneBauteile:TerminalBlock_MetzConnect_Type166x1x05_P3.50mm_Horizontal
- removed J91: Serial 1, TerminalBlock_MetzConnect:TerminalBlock_MetzConnect_Type059_RT06306HBWC_1x06_P3.50mm_Horizontal
- removed J92: Pullups´s, AA_EigeneBauteile:DIP-6_W7.62mm_SMD
- removed J94: +12V, AA_EigeneBauteile:TerminalBlock_MetzConnect_Type166_1x03_P3.50mm_Horizontal
- removed J96: LoRa, AA_EigeneBauteile:LoRa_Pinsocket_SMD
- removed R10, R11, R9: R LED, Resistor_SMD:R_0603_1608Metric_Pad0.98x0.95mm_HandSolder
- removed R5, R8: PULLUP, Resistor_SMD:R_0805_2012Metric_Pad1.20x1.40mm_HandSolder
- removed R6: R_Small, Resistor_SMD:R_0805_2012Metric_Pad1.20x1.40mm_HandSolder
- removed R7: Endwiderst. CAN, Resistor_SMD:R_0603_1608Metric_Pad0.98x0.95mm_HandSolder
- removed U12, U13: ULN2803A, AA_EigeneBauteile:DIP-18_W7.62mm_SMD
- added C2: 100nF, Capacitor_SMD:C_0805_2012Metric_Pad1.18x1.45mm_HandSolder, F.Cu at (216.3, 140.2)
- added R2: PULLUP, Resistor_SMD:R_0805_2012Metric_Pad1.20x1.40mm_HandSolder, F.Cu at (307.1, 101.5)
- C1: value 100nF -> C_Polarized; footprint Capacitor_SMD:C_0805_2012Metric_Pad1.18x1.45mm_HandSolder -> Capacitor_SMD:CP_Elec_4x5.4
- C4: value C -> 100nF; footprint Capacitor_THT:C_Disc_D3.0mm_W1.6mm_P2.50mm -> Capacitor_SMD:C_0805_2012Metric_Pad1.18x1.45mm_HandSolder
- J1: value GND +12V -> Spannungsversorgung +12V DC; footprint AA_EigeneBauteile:TerminalBlock_MetzConnect_Type166_1x02_P3.50mm_Horizontal -> TerminalBlock_MetzConnect:TerminalBlock_MetzConnect_Type011_RT05504HBWC_1x04_P5.00mm_Horizontal
- J10: value RJ45_LED_Shielded -> Serial 3; footprint Connector_RJ:RJ45_Cetus_J1B1211CCD_Horizontal -> TerminalBlock_MetzConnect:TerminalBlock_MetzConnect_Type011_RT05504HBWC_1x04_P5.00mm_Horizontal
- J11: value Serial 5 -> Serial 4; footprint TerminalBlock_MetzConnect:TerminalBlock_MetzConnect_Type059_RT06306HBWC_1x06_P3.50mm_Horizontal -> TerminalBlock_MetzConnect:TerminalBlock_MetzConnect_Type011_RT05504HBWC_1x04_P5.00mm_Horizontal
- J12: value Serial 6 -> Serial 5; footprint TerminalBlock_MetzConnect:TerminalBlock_MetzConnect_Type059_RT06306HBWC_1x06_P3.50mm_Horizontal -> TerminalBlock_MetzConnect:TerminalBlock_MetzConnect_Type011_RT05504HBWC_1x04_P5.00mm_Horizontal
- J13: value Serial 7 -> Serial 6; footprint TerminalBlock_MetzConnect:TerminalBlock_MetzConnect_Type059_RT06306HBWC_1x06_P3.50mm_Horizontal -> TerminalBlock_MetzConnect:TerminalBlock_MetzConnect_Type011_RT05504HBWC_1x04_P5.00mm_Horizontal
- J14: value Serial 8 -> I2C; footprint TerminalBlock_MetzConnect:TerminalBlock_MetzConnect_Type059_RT06306HBWC_1x06_P3.50mm_Horizontal -> TerminalBlock_MetzConnect:TerminalBlock_MetzConnect_Type011_RT05504HBWC_1x04_P5.00mm_Horizontal
- J15: value CAN 1 -> 1Wire; footprint TerminalBlock_MetzConnect:TerminalBlock_MetzConnect_Type059_RT06306HBWC_1x06_P3.50mm_Horizontal -> TerminalBlock_MetzConnect:TerminalBlock_MetzConnect_Type011_RT05504HBWC_1x04_P5.00mm_Horizontal
- J16, J41: value Conn_01x02 -> Digitale Eingänge; footprint AA_EigeneBauteile:TerminalBlock_MetzConnect_Type166_1x02_P3.50mm_Horizontal -> TerminalBlock_MetzConnect:TerminalBlock_MetzConnect_Type011_RT05502HBWC_1x02_P5.00mm_Horizontal
- J17, J18, J19, J20, J21, J22, J23, J24, J25, J26, J27, J28, J29, J30, J31, J34, J35, J36, J37, J38, J39, J42, J43, J44, J45, J46, J47, J48, J49, J50, J51, J52, J53, J54, J55, J56, J57, J60, J61, J62, J63, J64: value Conn_01x02 -> Conn_01x02_Male; footprint AA_EigeneBauteile:TerminalBlock_MetzConnect_Type166_1x02_P3.50mm_Horizontal -> TerminalBlock_MetzConnect:TerminalBlock_MetzConnect_Type011_RT05502HBWC_1x02_P5.00mm_Horizontal
- J2: value Conn_01x09 -> Spannungsversorgung GND; footprint AA_EigeneBauteile:PinSocket_1x9_P2.54mm_Vertical_SMD -> TerminalBlock_MetzConnect:TerminalBlock_MetzConnect_Type011_RT05504HBWC_1x04_P5.00mm_Horizontal
- J3: value Display128x64_I2C -> Conn_01x03_Female; footprint AA_EigeneBauteile:Display128x64_I2C_SMD -> Connector_PinSocket_2.54mm:PinSocket_1x03_P2.54mm_Vertical
- J32, J58: value +12V -> Conn_01x02_Male; footprint AA_EigeneBauteile:TerminalBlock_MetzConnect_Type166_1x03_P3.50mm_Horizontal -> TerminalBlock_MetzConnect:TerminalBlock_MetzConnect_Type011_RT05502HBWC_1x02_P5.00mm_Horizontal
- J33, J59: value GND -> Conn_01x02_Male; footprint AA_EigeneBauteile:TerminalBlock_MetzConnect_Type166_1x03_P3.50mm_Horizontal -> TerminalBlock_MetzConnect:TerminalBlock_MetzConnect_Type011_RT05502HBWC_1x02_P5.00mm_Horizontal
- J4: value +5V -> Conn_01x03_Female; footprint AA_EigeneBauteile:TerminalBlock_MetzConnect_Type166_1x03_P3.50mm_Horizontal -> Connector_PinSocket_2.54mm:PinSocket_1x03_P2.54mm_Vertical
- J40, J65: value Conn_01x02 -> Digitale Ausgänge; footprint AA_EigeneBauteile:TerminalBlock_MetzConnect_Type166_1x02_P3.50mm_Horizontal -> TerminalBlock_MetzConnect:TerminalBlock_MetzConnect_Type011_RT05502HBWC_1x02_P5.00mm_Horizontal
- J5: value Serial 2 -> Serial 1 - NFC-Reader 1; footprint TerminalBlock_MetzConnect:TerminalBlock_MetzConnect_Type059_RT06306HBWC_1x06_P3.50mm_Horizontal -> TerminalBlock_MetzConnect:TerminalBlock_MetzConnect_Type011_RT05504HBWC_1x04_P5.00mm_Horizontal
- J6: value Serial 3 -> I2C-Display; footprint TerminalBlock_MetzConnect:TerminalBlock_MetzConnect_Type059_RT06306HBWC_1x06_P3.50mm_Horizontal -> AA_EigeneBauteile:Display128x64_I2C
- J66: value Conn_01x02 -> Relais 1; footprint AA_EigeneBauteile:TerminalBlock_MetzConnect_Type166_1x02_P3.50mm_Horizontal -> TerminalBlock_MetzConnect:TerminalBlock_MetzConnect_Type055_RT01503HDWU_1x03_P5.00mm_Horizontal
- J67: value Conn_01x02 -> Relais 2; footprint AA_EigeneBauteile:TerminalBlock_MetzConnect_Type166_1x02_P3.50mm_Horizontal -> TerminalBlock_MetzConnect:TerminalBlock_MetzConnect_Type055_RT01503HDWU_1x03_P5.00mm_Horizontal
- J68: value Relais 1 -> Relais 3; footprint AA_EigeneBauteile:TerminalBlock_MetzConnect_Type166_1x03_P3.50mm_Horizontal -> TerminalBlock_MetzConnect:TerminalBlock_MetzConnect_Type055_RT01503HDWU_1x03_P5.00mm_Horizontal
- J69: value Relais 2 -> Relais 4; footprint AA_EigeneBauteile:TerminalBlock_MetzConnect_Type166_1x03_P3.50mm_Horizontal -> TerminalBlock_MetzConnect:TerminalBlock_MetzConnect_Type055_RT01503HDWU_1x03_P5.00mm_Horizontal
- J7: value Conn_01x24_Female -> Serial 2 - NFC-Reader 2; footprint AA_EigeneBauteile:PinSocket_1x24_P2.54mm_Vertical_SMD -> TerminalBlock_MetzConnect:TerminalBlock_MetzConnect_Type011_RT05504HBWC_1x04_P5.00mm_Horizontal
- J70: value Relais 3 -> Relais 5; footprint AA_EigeneBauteile:TerminalBlock_MetzConnect_Type166_1x03_P3.50mm_Horizontal -> TerminalBlock_MetzConnect:TerminalBlock_MetzConnect_Type055_RT01503HDWU_1x03_P5.00mm_Horizontal
- J71: value Relais 4 -> Relais 6; footprint AA_EigeneBauteile:TerminalBlock_MetzConnect_Type166_1x03_P3.50mm_Horizontal -> TerminalBlock_MetzConnect:TerminalBlock_MetzConnect_Type055_RT01503HDWU_1x03_P5.00mm_Horizontal
- J72: value Relais 5 -> Relais 7; footprint AA_EigeneBauteile:TerminalBlock_MetzConnect_Type166_1x03_P3.50mm_Horizontal -> TerminalBlock_MetzConnect:TerminalBlock_MetzConnect_Type055_RT01503HDWU_1x03_P5.00mm_Horizontal
- J73: value Relais 6 -> Relais 8; footprint AA_EigeneBauteile:TerminalBlock_MetzConnect_Type166_1x03_P3.50mm_Horizontal -> TerminalBlock_MetzConnect:TerminalBlock_MetzConnect_Type055_RT01503HDWU_1x03_P5.00mm_Horizontal
- J8: footprint AA_EigeneBauteile:PinSocket_1x24_P2.54mm_Vertical_SMD -> Connector_PinSocket_2.54mm:PinSocket_1x24_P2.54mm_Vertical
- J9: value Serial 4 -> Conn_01x24_Female; footprint TerminalBlock_MetzConnect:TerminalBlock_MetzConnect_Type059_RT06306HBWC_1x06_P3.50mm_Horizontal -> Connector_PinSocket_2.54mm:PinSocket_1x24_P2.54mm_Vertical
- R1: value Endwiderst. CAN -> R_Small; footprint Resistor_SMD:R_0603_1608Metric_Pad0.98x0.95mm_HandSolder -> Resistor_SMD:R_0805_2012Metric_Pad1.20x1.40mm_HandSolder
- R3: value R_Small -> PULLUP
- R4: value PULLUP -> R_Small
- RN1, RN2, RN3, RN4, RN5: footprint AA_EigeneBauteile:PinSocket_1x9_P2.54mm_Vertical_SMD -> Resistor_THT:R_Array_SIP9
- U1: value OKI-78SR-3.3_1.5-W36-C -> OKI-78SR-5_1.5-W36-C
- U10, U6: value MCP23S17_SP -> ULN2803A; footprint AA_EigeneBauteile:DIP-28_W7.62mm_SMD -> AA_EigeneBauteile:DIP-18_W7.62mm_SMD
- U11, U7: value MCP23017_SP -> ULN2803A; footprint AA_EigeneBauteile:DIP-28_W7.62mm_SMD -> AA_EigeneBauteile:DIP-18_W7.62mm_SMD
- U2: value OKI-78SR-5_1.5-W36-C -> Teensy4.1; footprint Converter_DCDC:Converter_DCDC_Murata_OKI-78SR_Vertical -> teensy:Teensy41
- U3: value Teensy4.1 -> ULN2803A; footprint AA_EigeneBauteile:Teensy41_without_some_pins_SMD -> AA_EigeneBauteile:DIP-18_W7.62mm_SMD
- U5, U9: value ULN2803A -> MCP23017_SP; footprint AA_EigeneBauteile:DIP-18_W7.62mm_SMD -> AA_EigeneBauteile:DIP-28_W7.62mm_SMD
- U8: value ULN2803A -> MCP23S17_SP; footprint AA_EigeneBauteile:DIP-18_W7.62mm_SMD -> AA_EigeneBauteile:DIP-28_W7.62mm_SMD
- moved J66 273.5 mm to (95.7, 248.2)
- moved J67 266.8 mm to (112.2, 248.2)
- moved J41 261.3 mm to (72.8, 71.7), turned to 180 degrees
- moved R3 233.4 mm to (307.7, 219.0)
- moved U7 209.4 mm to (284.9, 186.6)
- moved J10 204.7 mm to (70.9, 155.0), turned to -90 degrees
- moved J4 193.1 mm to (123.6, 165.0), turned to 90 degrees
- moved R1 187.4 mm to (201.1, 43.1), turned to 90 degrees
- moved J2 162.7 mm to (337.1, 246.9), turned to 0 degrees
- moved U2 160.8 mm to (183.3, 132.0), turned to 180 degrees
- moved U8 160.7 mm to (284.9, 219.0)
- moved J7 159.1 mm to (70.9, 129.6)
- moved U11 156.6 mm to (226.4, 206.9), turned to -90 degrees
- moved C6 155.5 mm to (289.9, 229.1), turned to 0 degrees
- moved SW1 155.1 mm to (249.3, 252.5)
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Connections:
- C1 pad 1: +3.3V -> +5V
- C3 pad 1: +5V -> 3,3V
- C4 pad 1: Net-(C4-Pad1) -> 3,3V
- C4 pad 2: Net-(C4-Pad2) -> GND
- C5 pad 1: +3.3V -> 3,3V
- C6 pad 1: +3.3V -> 3,3V
- D1 pad 1: Net-(D1-K) -> Net-(D1-Pad1)
- D10 pad 1: Net-(D10-K) -> Net-(D10-Pad1)
- D11 pad 1: Net-(D11-K) -> Net-(D11-Pad1)
- D12 pad 1: Net-(D12-K) -> Net-(D12-Pad1)
- D13 pad 1: Net-(D13-K) -> Net-(D13-Pad1)
- D14 pad 1: Net-(D14-K) -> Net-(D14-Pad1)
- D15 pad 1: Net-(D15-K) -> Net-(D15-Pad1)
- D16 pad 1: Net-(D16-K) -> Net-(D16-Pad1)
- D17 pad 1: Net-(D17-K) -> Net-(D17-Pad1)
- D18 pad 1: Net-(D18-K) -> Net-(D18-Pad1)
- D19 pad 1: Net-(D19-K) -> Net-(D19-Pad1)
- D2 pad 1: Net-(D2-K) -> Net-(D2-Pad1)
- D20 pad 1: Net-(D20-K) -> Net-(D20-Pad1)
- D21 pad 1: Net-(D21-K) -> Net-(D21-Pad1)
- D22 pad 1: Net-(D22-K) -> Net-(D22-Pad1)
- D23 pad 1: Net-(D23-K) -> Net-(D23-Pad1)
- D24 pad 1: Net-(D24-K) -> Net-(D24-Pad1)
- D25 pad 1: Net-(D25-K) -> Net-(D25-Pad1)
- D26 pad 1: Net-(D26-K) -> Net-(D26-Pad1)
- D27 pad 1: Net-(D27-K) -> Net-(D27-Pad1)
- D28 pad 1: Net-(D28-K) -> Net-(D28-Pad1)
- D29 pad 1: Net-(D29-K) -> Net-(D29-Pad1)
- D3 pad 1: Net-(D3-K) -> Net-(D3-Pad1)
- D30 pad 1: Net-(D30-K) -> Net-(D30-Pad1)
- D31 pad 1: Net-(D31-K) -> Net-(D31-Pad1)
- D32 pad 1: Net-(D32-K) -> Net-(D32-Pad1)
- D33 pad 1: Net-(D33-K) -> Net-(D33-Pad1)
- D34 pad 1: Net-(D34-K) -> Net-(D34-Pad1)
- D35 pad 1: Net-(D35-K) -> Net-(D35-Pad1)
- D36 pad 1: Net-(D36-K) -> Net-(D36-Pad1)
- D37 pad 1: Net-(D37-K) -> Net-(D37-Pad1)
- D38 pad 1: Net-(D38-K) -> Net-(D38-Pad1)
- D39 pad 1: Net-(D39-K) -> Net-(D39-Pad1)
- D4 pad 1: Net-(D4-K) -> Net-(D4-Pad1)
- D40 pad 1: Net-(D40-K) -> Net-(D40-Pad1)
- D5 pad 1: Net-(D5-K) -> Net-(D5-Pad1)
- D6 pad 1: Net-(D6-K) -> Net-(D6-Pad1)
- D7 pad 1: Net-(D7-K) -> Net-(D7-Pad1)
- D8 pad 1: Net-(D8-K) -> Net-(D8-Pad1)
- D9 pad 1: Net-(D9-K) -> Net-(D9-Pad1)
- J1 pad 1: GND -> +12V
- J10 pad 1: Net-(U3-T+) -> 3,3V
- J10 pad 2: Net-(C4-Pad2) -> GND
- J10 pad 3: Net-(U3-T-) -> RX3
- J10 pad 4: Net-(U3-R+) -> TX3
- J11 pad 1: RX5 -> 3,3V
- J11 pad 2: TX5 -> GND
- J11 pad 3: +12V.1 -> RX4
- J11 pad 4: +5V -> TX4
- J12 pad 1: RX6 -> 3,3V
- J12 pad 2: TX6 -> GND
- J12 pad 3: +12V.1 -> RX5
- J12 pad 4: +5V -> TX5
- J13 pad 1: RX7 -> 3,3V
- J13 pad 2: TX7 -> GND
- J13 pad 3: +12V.1 -> RX6
- J13 pad 4: +5V -> TX6
- J14 pad 1: RX8 -> 3,3V
- J14 pad 2: TX8 -> GND
- J14 pad 3: +12V.1 -> SDA
- J14 pad 4: +5V -> SCL
- J15 pad 1: Net-(J15-Pin_1) -> 3,3V
- J15 pad 2: Net-(J15-Pin_2) -> GND
- J15 pad 3: +12V.1 -> 1Wire
- J15 pad 4: +5V -> unconnected-(J15-Pad4)
- J16 pad 1: Net-(J16-Pin_1) -> Net-(J16-Pad1)
- J17 pad 1: Net-(J17-Pin_1) -> Net-(J17-Pad1)
- J18 pad 1: Net-(J18-Pin_1) -> Net-(J18-Pad1)
- J19 pad 1: Net-(J19-Pin_1) -> Net-(J19-Pad1)
- J2 pad 1: Net-(J2-Pin_1) -> GND
- J2 pad 2: Net-(J2-Pin_2) -> GND
- J2 pad 3: Net-(J2-Pin_3) -> GND
- J2 pad 4: Net-(J2-Pin_4) -> GND
- J20 pad 1: Net-(J20-Pin_1) -> Net-(J20-Pad1)
- J21 pad 1: Net-(J21-Pin_1) -> Net-(J21-Pad1)
- J22 pad 1: Net-(J22-Pin_1) -> Net-(J22-Pad1)
- J23 pad 1: Net-(J23-Pin_1) -> Net-(J23-Pad1)
- J24 pad 1: Net-(J24-Pin_1) -> Net-(J24-Pad1)
- J25 pad 1: Net-(J25-Pin_1) -> Net-(J25-Pad1)
- J26 pad 1: Net-(J26-Pin_1) -> Net-(J26-Pad1)
- J27 pad 1: Net-(J27-Pin_1) -> Net-(J27-Pad1)
- J28 pad 1: Net-(J28-Pin_1) -> Net-(J28-Pad1)
- J29 pad 1: Net-(J29-Pin_1) -> Net-(J29-Pad1)
- J3 pad 1: +3.3V -> 3,3V
- J3 pad 2: GND -> 3,3V
- J3 pad 3: SCL -> 3,3V
- J30 pad 1: Net-(J30-Pin_1) -> Net-(J30-Pad1)
- J31 pad 1: Net-(J31-Pin_1) -> Net-(J31-Pad1)
- J32 pad 1: +12V.1 -> +12V
- J32 pad 2: +12V.1 -> +12V
- J33 pad 1: GND -> Net-(D2-Pad1)
- J33 pad 2: GND -> Net-(D1-Pad1)
- J34 pad 1: Net-(D1-K) -> Net-(D4-Pad1)
- J34 pad 2: Net-(D2-K) -> Net-(D3-Pad1)
- J35 pad 1: Net-(D3-K) -> Net-(D6-Pad1)
- J35 pad 2: Net-(D4-K) -> Net-(D5-Pad1)
- J36 pad 1: Net-(D5-K) -> Net-(D8-Pad1)
- J36 pad 2: Net-(D6-K) -> Net-(D7-Pad1)
- J37 pad 1: Net-(D7-K) -> Net-(D10-Pad1)
- J37 pad 2: Net-(D8-K) -> Net-(D9-Pad1)
- J38 pad 1: Net-(D9-K) -> Net-(D12-Pad1)
- J38 pad 2: Net-(D10-K) -> Net-(D11-Pad1)
- J39 pad 1: Net-(D11-K) -> Net-(D14-Pad1)
- J39 pad 2: Net-(D12-K) -> Net-(D13-Pad1)
- J4 pad 1: +5V -> 1Wire
- J4 pad 2: +5V -> SDA
- J4 pad 3: +5V -> SCL
- J40 pad 1: Net-(D13-K) -> Net-(D16-Pad1)
- J40 pad 2: Net-(D14-K) -> Net-(D15-Pad1)
- J41 pad 1: Net-(D15-K) -> Net-(J41-Pad1)
- J41 pad 2: Net-(D16-K) -> GND
- J42 pad 1: Net-(J42-Pin_1) -> Net-(J42-Pad1)
- J43 pad 1: Net-(J43-Pin_1) -> Net-(J43-Pad1)
- J44 pad 1: Net-(J44-Pin_1) -> Net-(J44-Pad1)
- J45 pad 1: Net-(J45-Pin_1) -> Net-(J45-Pad1)
- J46 pad 1: Net-(J46-Pin_1) -> Net-(J46-Pad1)
- J47 pad 1: Net-(J47-Pin_1) -> Net-(J47-Pad1)
- J48 pad 1: Net-(J48-Pin_1) -> Net-(J48-Pad1)
- J49 pad 1: Net-(J49-Pin_1) -> Net-(J49-Pad1)
- J5 pad 1: RX2 -> 3,3V
- J5 pad 2: TX2 -> GND
- J5 pad 3: +12V.1 -> RX1
- J5 pad 4: +5V -> TX1
- J50 pad 1: Net-(J50-Pin_1) -> Net-(J50-Pad1)
- J51 pad 1: Net-(J51-Pin_1) -> Net-(J51-Pad1)
- J52 pad 1: Net-(J52-Pin_1) -> Net-(J52-Pad1)
- J53 pad 1: Net-(J53-Pin_1) -> Net-(J53-Pad1)
- J54 pad 1: Net-(J54-Pin_1) -> Net-(J54-Pad1)
- J55 pad 1: Net-(J55-Pin_1) -> Net-(J55-Pad1)
- J56 pad 1: Net-(J56-Pin_1) -> Net-(J56-Pad1)
- J57 pad 1: Net-(J57-Pin_1) -> +12V
- J57 pad 2: GND -> +12V
- J58 pad 1: +12V.1 -> Net-(D18-Pad1)
- J58 pad 2: +12V.1 -> Net-(D17-Pad1)
- J59 pad 1: GND -> Net-(D20-Pad1)
- J59 pad 2: GND -> Net-(D19-Pad1)
- J6 pad 1: RX3 -> 3,3V
- J6 pad 2: TX3 -> GND
- J6 pad 3: +12V.1 -> SCL
- J6 pad 4: +5V -> SDA
- J60 pad 1: Net-(D17-K) -> Net-(D22-Pad1)
- J60 pad 2: Net-(D18-K) -> Net-(D21-Pad1)
- J61 pad 1: Net-(D19-K) -> Net-(D24-Pad1)
- J61 pad 2: Net-(D20-K) -> Net-(D23-Pad1)
- J62 pad 1: Net-(D21-K) -> Net-(D26-Pad1)
- J62 pad 2: Net-(D22-K) -> Net-(D25-Pad1)
- J63 pad 1: Net-(D23-K) -> Net-(D28-Pad1)
- J63 pad 2: Net-(D24-K) -> Net-(D27-Pad1)
- J64 pad 1: Net-(D25-K) -> Net-(D30-Pad1)
- J64 pad 2: Net-(D26-K) -> Net-(D29-Pad1)
- J65 pad 1: Net-(D27-K) -> Net-(D32-Pad1)
- J65 pad 2: Net-(D28-K) -> Net-(D31-Pad1)
- J66 pad 1: Net-(D29-K) -> Net-(J66-Pad1)
- J66 pad 2: Net-(D30-K) -> Net-(J66-Pad2)
- J67 pad 1: Net-(D31-K) -> Net-(J67-Pad1)
- J67 pad 2: Net-(D32-K) -> Net-(J67-Pad2)
- J68 pad 1: Net-(J68-Pin_1) -> Net-(J68-Pad1)
- J68 pad 2: Net-(J68-Pin_2) -> Net-(J68-Pad2)
- J68 pad 3: Net-(J68-Pin_3) -> Net-(J68-Pad3)
- J69 pad 1: Net-(J69-Pin_1) -> Net-(J69-Pad1)
- J69 pad 2: Net-(J69-Pin_2) -> Net-(J69-Pad2)
- J69 pad 3: Net-(J69-Pin_3) -> Net-(J69-Pad3)
- J7 pad 1: GND -> 3,3V
- J7 pad 2: RX1 -> GND
- J7 pad 3: TX1 -> RX2
- J7 pad 4: Taster -> TX2
- J70 pad 1: Net-(J70-Pin_1) -> Net-(J70-Pad1)
- J70 pad 2: Net-(J70-Pin_2) -> Net-(J70-Pad2)
- J70 pad 3: Net-(J70-Pin_3) -> Net-(J70-Pad3)
- J71 pad 1: Net-(J71-Pin_1) -> Net-(J71-Pad1)
- J71 pad 2: Net-(J71-Pin_2) -> Net-(J71-Pad2)
- J71 pad 3: Net-(J71-Pin_3) -> Net-(J71-Pad3)
- J72 pad 1: Net-(J72-Pin_1) -> Net-(J72-Pad1)
- J72 pad 2: Net-(J72-Pin_2) -> Net-(J72-Pad2)
- J72 pad 3: Net-(J72-Pin_3) -> Net-(J72-Pad3)
- J73 pad 1: Net-(J73-Pin_1) -> Net-(J73-Pad1)
- J73 pad 2: Net-(J73-Pin_2) -> Net-(J73-Pad2)
- J73 pad 3: Net-(J73-Pin_3) -> Net-(J73-Pad3)
- J8 pad 1: +5V -> GND
- J8 pad 10: TX4 -> TX2
- J8 pad 11: RX4 -> Net-(J8-Pad11)
- J8 pad 12: RX3 -> Net-(J8-Pad12)
- J8 pad 13: TX3 -> 1Wire
- J8 pad 14: Net-(J8-Pin_14) -> Net-(J8-Pad14)
- J8 pad 15: GND -> Net-(J8-Pad15)
- J8 pad 16: LoRa_IRQ -> TX6
- J8 pad 17: LoRa_Reset -> RX6
- J8 pad 18: SPI_MISO1 -> Net-(J8-Pad18)
- J8 pad 19: SPI_CS1 -> Net-(J8-Pad19)
- J8 pad 2: GND -> RX1
- J8 pad 20: SPI_SCK -> Net-(J8-Pad20)
- J8 pad 21: Net-(J8-Pin_21) -> Net-(J8-Pad21)
- J8 pad 22: TX8 -> Net-(J8-Pad22)
- J8 pad 23: RX8 -> Net-(J8-Pad23)
- J8 pad 24: Relais1 -> Net-(J8-Pad24)
- J8 pad 3: Net-(J8-Pin_3) -> TX1
- J8 pad 4: CAN1_RX -> Net-(J8-Pad4)
- J8 pad 5: CAN1_TX -> Net-(J8-Pad5)
- J8 pad 6: RX5 -> Net-(J8-Pad6)
- J8 pad 7: TX5 -> Net-(J8-Pad7)
- J8 pad 8: SCL -> Net-(J8-Pad8)
- J8 pad 9: SDA -> RX2
- J9 pad 1: RX4 -> +5V
- J9 pad 2: TX4 -> GND
- J9 pad 3: +12V.1 -> 3,3V
- J9 pad 4: +5V -> Net-(J9-Pad4)
- J9 pad 5: +3.3V -> Net-(J9-Pad5)
- J9 pad 6: GND -> RX5
- K1 pad 11: Net-(J68-Pin_2) -> Net-(J66-Pad2)
- K1 pad 12: Net-(J68-Pin_3) -> Net-(J66-Pad3)
- K1 pad 14: Net-(J68-Pin_1) -> Net-(J66-Pad1)
- K1 pad A1: Net-(D33-K) -> Net-(D33-Pad1)
- K1 pad A2: +12V.1 -> +12V
- K2 pad 11: Net-(J69-Pin_2) -> Net-(J67-Pad2)
- K2 pad 12: Net-(J69-Pin_3) -> Net-(J67-Pad3)
- K2 pad 14: Net-(J69-Pin_1) -> Net-(J67-Pad1)
- K2 pad A1: Net-(D34-K) -> Net-(D34-Pad1)
- K2 pad A2: +12V.1 -> +12V
- K3 pad 11: Net-(J70-Pin_2) -> Net-(J68-Pad2)
- K3 pad 12: Net-(J70-Pin_3) -> Net-(J68-Pad3)
- K3 pad 14: Net-(J70-Pin_1) -> Net-(J68-Pad1)
- K3 pad A1: Net-(D35-K) -> Net-(D35-Pad1)
- K3 pad A2: +12V.1 -> +12V
- K4 pad 11: Net-(J71-Pin_2) -> Net-(J69-Pad2)
- K4 pad 12: Net-(J71-Pin_3) -> Net-(J69-Pad3)
- K4 pad 14: Net-(J71-Pin_1) -> Net-(J69-Pad1)
- K4 pad A1: Net-(D36-K) -> Net-(D36-Pad1)
- K4 pad A2: +12V.1 -> +12V
- K5 pad 11: Net-(J72-Pin_2) -> Net-(J70-Pad2)
- K5 pad 12: Net-(J72-Pin_3) -> Net-(J70-Pad3)
- K5 pad 14: Net-(J72-Pin_1) -> Net-(J70-Pad1)
- K5 pad A1: Net-(D37-K) -> Net-(D37-Pad1)
- K5 pad A2: +12V.1 -> +12V
- K6 pad 11: Net-(J73-Pin_2) -> Net-(J71-Pad2)
- K6 pad 12: Net-(J73-Pin_3) -> Net-(J71-Pad3)
- K6 pad 14: Net-(J73-Pin_1) -> Net-(J71-Pad1)
- K6 pad A1: Net-(D38-K) -> Net-(D38-Pad1)
- K6 pad A2: +12V.1 -> +12V
- K7 pad 11: Net-(J74-Pin_2) -> Net-(J72-Pad2)
- K7 pad 12: Net-(J74-Pin_3) -> Net-(J72-Pad3)
- K7 pad 14: Net-(J74-Pin_1) -> Net-(J72-Pad1)
- K7 pad A1: Net-(D39-K) -> Net-(D39-Pad1)
- K7 pad A2: +12V.1 -> +12V
- K8 pad 11: Net-(J75-Pin_2) -> Net-(J73-Pad2)
- K8 pad 12: Net-(J75-Pin_3) -> Net-(J73-Pad3)
- K8 pad 14: Net-(J75-Pin_1) -> Net-(J73-Pad1)
- K8 pad A1: Net-(D40-K) -> Net-(D40-Pad1)
- K8 pad A2: +12V.1 -> +12V
- R1 pad 1: Net-(J87-Pin_2) -> 3,3V
- R1 pad 2: Net-(J15-Pin_1) -> Net-(R1-Pad2)
- R3 pad 1: +3.3V -> 3,3V
- R3 pad 2: Net-(U7-~{RESET}) -> Net-(R3-Pad2)
- R4 pad 1: +3.3V -> 3,3V
- R4 pad 2: Net-(U6-~{RESET}) -> Net-(R4-Pad2)
- RN1 pad 1: +12V.1 -> +12V
- RN2 pad 1: +12V.1 -> +12V
- RN3 pad 1: +12V.1 -> +12V
- RN4 pad 1: +12V.1 -> +12V
- RN5 pad 1: +12V.1 -> +12V
- U1 pad 1: Net-(U1-IN) -> +12V
- U1 pad 3: Net-(U1-OUT) -> +5V
- U10 pad 1: Net-(U10-GPB0) -> Net-(U10-Pad1)
- U10 pad 10: GND -> +12V
- U10 pad 11: unconnected-(U10-NC-Pad11) -> Net-(D32-Pad1)
- U10 pad 12: SCL -> Net-(D31-Pad1)
- U10 pad 13: SDA -> Net-(D30-Pad1)
- U10 pad 14: unconnected-(U10-NC-Pad14) -> Net-(D29-Pad1)
- U10 pad 15: +3.3V -> Net-(D28-Pad1)
- U10 pad 16: +3.3V -> Net-(D27-Pad1)
- U10 pad 17: GND -> Net-(D26-Pad1)
- U10 pad 18: Net-(U10-~{RESET}) -> Net-(D25-Pad1)
- U10 pad 2: Net-(U10-GPB1) -> Net-(U10-Pad2)
- U10 pad 3: Net-(U10-GPB2) -> Net-(U10-Pad3)
- U10 pad 4: Net-(U10-GPB3) -> Net-(U10-Pad4)
- U10 pad 5: Net-(U10-GPB4) -> Net-(U10-Pad5)
- U10 pad 6: Net-(U10-GPB5) -> Net-(U10-Pad6)
- U10 pad 7: Net-(U10-GPB6) -> Net-(U10-Pad7)
- U10 pad 8: Net-(U10-GPB7) -> Net-(U10-Pad8)
- U10 pad 9: +3.3V -> GND
- U11 pad 1: Net-(J42-Pin_1) -> Relais 1
- U11 pad 10: GND -> +12V
- U11 pad 11: unconnected-(U11-NC-Pad11) -> Net-(D40-Pad1)
- U11 pad 12: SCL -> Net-(D39-Pad1)
- U11 pad 13: SDA -> Net-(D38-Pad1)
- U11 pad 14: unconnected-(U11-NC-Pad14) -> Net-(D37-Pad1)
- U11 pad 15: +3.3V -> Net-(D36-Pad1)
- U11 pad 16: GND -> Net-(D35-Pad1)
- U11 pad 17: GND -> Net-(D34-Pad1)
- U11 pad 18: Net-(U11-~{RESET}) -> Net-(D33-Pad1)
- U11 pad 2: Net-(J43-Pin_1) -> Relais 2
- U11 pad 3: Net-(J44-Pin_1) -> Relais 3
- U11 pad 4: Net-(J45-Pin_1) -> Relais 4
- U11 pad 5: Net-(J46-Pin_1) -> Relais 5
- U11 pad 6: Net-(J47-Pin_1) -> Relais 6
- U11 pad 7: Net-(J48-Pin_1) -> Relais 7
- U11 pad 8: Net-(J49-Pin_1) -> Relais 8
- U11 pad 9: +3.3V -> GND
- U2 pad 1: +12V -> GND
- U2 pad 2: GND -> RX1
- U2 pad 3: Net-(U1-IN) -> TX1
- U3 pad 1: GND -> Net-(U3-Pad1)
- U3 pad 10: TX2 -> +12V
- U3 pad 11: 1Wire -> Net-(D8-Pad1)
- U3 pad 12: SPI_CS -> Net-(D7-Pad1)
- U3 pad 13: SPI_MOSI -> Net-(D6-Pad1)
- U3 pad 14: SPI_MISO -> Net-(D5-Pad1)
- U3 pad 15: Net-(J7-Pin_15) -> Net-(D4-Pad1)
- U3 pad 16: TX6 -> Net-(D3-Pad1)
- U3 pad 17: RX6 -> Net-(D2-Pad1)
- U3 pad 18: SPI_MOSI1 -> Net-(D1-Pad1)
- U3 pad 2: RX1 -> Net-(U3-Pad2)
- U3 pad 3: TX1 -> Net-(U3-Pad3)
- U3 pad 4: Taster -> Net-(U3-Pad4)
- U3 pad 5: MCP0_INTB -> Net-(U3-Pad5)
- U3 pad 6: MCP0_INTA -> Net-(U3-Pad6)
- U3 pad 7: MCP1_INTA -> Net-(U3-Pad7)
- U3 pad 8: MCP1_INTB -> Net-(U3-Pad8)
- U3 pad 9: RX2 -> GND
- U4 pad 1: Net-(U13-I8) -> Net-(U3-Pad1)
- U4 pad 15: +3.3V -> GND
- U4 pad 16: +3.3V -> 3,3V
- U4 pad 17: +3.3V -> GND
- U4 pad 2: Net-(U13-I7) -> Net-(U3-Pad2)
- U4 pad 21: Net-(J2-Pin_1) -> Net-(U4-Pad21)
- U4 pad 22: Net-(J2-Pin_2) -> Net-(U4-Pad22)
- U4 pad 23: Net-(J2-Pin_3) -> Net-(U4-Pad23)
- U4 pad 24: Net-(J2-Pin_4) -> Net-(U4-Pad24)
- U4 pad 25: Net-(J2-Pin_5) -> Net-(U4-Pad25)
- U4 pad 26: Net-(J2-Pin_6) -> Net-(U4-Pad26)
- U4 pad 27: Net-(J2-Pin_7) -> Net-(U4-Pad27)
- U4 pad 28: Net-(J2-Pin_8) -> Net-(U4-Pad28)
- U4 pad 3: Net-(U13-I6) -> Net-(U3-Pad3)
- U4 pad 4: Net-(U13-I5) -> Net-(U3-Pad4)
- U4 pad 5: Net-(U13-I4) -> Net-(U3-Pad5)
- U4 pad 6: Net-(U13-I3) -> Net-(U3-Pad6)
- U4 pad 7: Net-(U13-I2) -> Net-(U3-Pad7)
- U4 pad 8: Net-(U13-I1) -> Net-(U3-Pad8)
- U4 pad 9: +3.3V -> 3,3V
- U5 pad 1: Net-(U5-I1) -> Net-(J16-Pad1)
- U5 pad 10: +12V.1 -> GND
- U5 pad 11: Net-(D8-K) -> unconnected-(U5-Pad11)
- U5 pad 12: Net-(D7-K) -> SCL
- U5 pad 13: Net-(D6-K) -> SDA
- U5 pad 14: Net-(D5-K) -> unconnected-(U5-Pad14)
- U5 pad 15: Net-(D4-K) -> GND
- U5 pad 16: Net-(D3-K) -> GND
- U5 pad 17: Net-(D2-K) -> GND
- U5 pad 18: Net-(D1-K) -> Net-(R1-Pad2)
- U5 pad 2: Net-(U5-I2) -> Net-(J17-Pad1)
- U5 pad 3: Net-(U5-I3) -> Net-(J18-Pad1)
- U5 pad 4: Net-(U5-I4) -> Net-(J19-Pad1)
- U5 pad 5: Net-(U5-I5) -> Net-(J20-Pad1)
- U5 pad 6: Net-(U5-I6) -> Net-(J21-Pad1)
- U5 pad 7: Net-(U5-I7) -> Net-(J22-Pad1)
- U5 pad 8: Net-(U5-I8) -> Net-(J23-Pad1)
- U5 pad 9: GND -> 3,3V
- U6 pad 1: Net-(U5-I1) -> Net-(U4-Pad21)
- U6 pad 10: GND -> +12V
- U6 pad 11: unconnected-(U6-NC-Pad11) -> Net-(D16-Pad1)
- U6 pad 12: SCL -> Net-(D15-Pad1)
- U6 pad 13: SDA -> Net-(D14-Pad1)
- U6 pad 14: unconnected-(U6-NC-Pad14) -> Net-(D13-Pad1)
- U6 pad 15: GND -> Net-(D12-Pad1)
- U6 pad 16: +3.3V -> Net-(D11-Pad1)
- U6 pad 17: GND -> Net-(D10-Pad1)
- U6 pad 18: Net-(U6-~{RESET}) -> Net-(D9-Pad1)
- U6 pad 2: Net-(U5-I2) -> Net-(U4-Pad22)
- U6 pad 3: Net-(U5-I3) -> Net-(U4-Pad23)
- U6 pad 4: Net-(U5-I4) -> Net-(U4-Pad24)
- U6 pad 5: Net-(U5-I5) -> Net-(U4-Pad25)
- U6 pad 6: Net-(U5-I6) -> Net-(U4-Pad26)
- U6 pad 7: Net-(U5-I7) -> Net-(U4-Pad27)
- U6 pad 8: Net-(U5-I8) -> Net-(U4-Pad28)
- U6 pad 9: +3.3V -> GND
- U7 pad 1: Net-(J16-Pin_1) -> Net-(U7-Pad1)
- U7 pad 10: GND -> +12V
- U7 pad 11: unconnected-(U7-NC-Pad11) -> Net-(D24-Pad1)
- U7 pad 12: SCL -> Net-(D23-Pad1)
- U7 pad 13: SDA -> Net-(D22-Pad1)
- U7 pad 14: unconnected-(U7-NC-Pad14) -> Net-(D21-Pad1)
- U7 pad 15: GND -> Net-(D20-Pad1)
- U7 pad 16: GND -> Net-(D19-Pad1)
- U7 pad 17: GND -> Net-(D18-Pad1)
- U7 pad 18: Net-(U7-~{RESET}) -> Net-(D17-Pad1)
- U7 pad 2: Net-(J17-Pin_1) -> Net-(U7-Pad2)
- U7 pad 3: Net-(J18-Pin_1) -> Net-(U7-Pad3)
- U7 pad 4: Net-(J19-Pin_1) -> Net-(U7-Pad4)
- U7 pad 5: Net-(J20-Pin_1) -> Net-(U7-Pad5)
- U7 pad 6: Net-(J21-Pin_1) -> Net-(U7-Pad6)
- U7 pad 7: Net-(J22-Pin_1) -> Net-(U7-Pad7)
- U7 pad 8: Net-(J23-Pin_1) -> Net-(U7-Pad8)
- U7 pad 9: +3.3V -> GND
- U8 pad 1: Net-(U6-GPA0) -> Net-(U7-Pad1)
- U8 pad 10: +12V.1 -> GND
- U8 pad 11: Net-(D16-K) -> unconnected-(U8-Pad11)
- U8 pad 12: Net-(D15-K) -> SCL
- U8 pad 13: Net-(D14-K) -> SDA
- U8 pad 14: Net-(D13-K) -> unconnected-(U8-Pad14)
- U8 pad 15: Net-(D12-K) -> 3,3V
- U8 pad 16: Net-(D11-K) -> 3,3V
- U8 pad 17: Net-(D10-K) -> GND
- U8 pad 18: Net-(D9-K) -> Net-(R3-Pad2)
- U8 pad 2: Net-(U6-GPA1) -> Net-(U7-Pad2)
- U8 pad 3: Net-(U6-GPA2) -> Net-(U7-Pad3)
- U8 pad 4: Net-(U6-GPA3) -> Net-(U7-Pad4)
- U8 pad 5: Net-(U6-GPA4) -> Net-(U7-Pad5)
- U8 pad 6: Net-(U6-GPA5) -> Net-(U7-Pad6)
- U8 pad 7: Net-(U6-GPA6) -> Net-(U7-Pad7)
- U8 pad 8: Net-(U6-GPA7) -> Net-(U7-Pad8)
- U8 pad 9: GND -> 3,3V
- U9 pad 1: Net-(U10-GPB0) -> Net-(J41-Pad1)
- U9 pad 10: +12V.1 -> GND
- U9 pad 11: Net-(D24-K) -> unconnected-(U9-Pad11)
- U9 pad 12: Net-(D23-K) -> SCL
- U9 pad 13: Net-(D22-K) -> SDA
- U9 pad 14: Net-(D21-K) -> unconnected-(U9-Pad14)
- U9 pad 15: Net-(D20-K) -> 3,3V
- U9 pad 16: Net-(D19-K) -> GND
- U9 pad 17: Net-(D18-K) -> GND
- U9 pad 18: Net-(D17-K) -> Net-(R4-Pad2)
- U9 pad 2: Net-(U10-GPB1) -> Net-(J42-Pad1)
- U9 pad 3: Net-(U10-GPB2) -> Net-(J43-Pad1)
- U9 pad 4: Net-(U10-GPB3) -> Net-(J44-Pad1)
- U9 pad 5: Net-(U10-GPB4) -> Net-(J45-Pad1)
- U9 pad 6: Net-(U10-GPB5) -> Net-(J46-Pad1)
- U9 pad 7: Net-(U10-GPB6) -> Net-(J47-Pad1)
- U9 pad 8: Net-(U10-GPB7) -> Net-(J48-Pad1)
- U9 pad 9: GND -> 3,3V
Routing:
- net +3.3V: track 1532.4 -> 0.00 mm, vias 6 -> 0
- net +12V.1: track 1253.1 -> 0.00 mm
- net 3,3V: track 0.00 -> 966.8 mm, vias 0 -> 5
- net +5V: track 866.4 -> 205.6 mm, vias 1 -> 0
- net +12V: track 64.2 -> 686.1 mm
- net SDA: track 374.6 -> 622.7 mm, vias 8 -> 6
- net SCL: track 381.1 -> 620.2 mm, vias 9 -> 5
- net Net-(D33-Pad1): track 0.00 -> 159.6 mm, vias 0 -> 1
- net CAN1_RX: track 153.8 -> 0.00 mm, vias 3 -> 0
- net CAN1_TX: track 149.0 -> 0.00 mm, vias 3 -> 0
- net Relais 1: track 0.00 -> 142.7 mm, vias 0 -> 1
- net Net-(C4-Pad1): track 141.4 -> 0.00 mm, vias 3 -> 0
- net Relais 2: track 0.00 -> 140.0 mm, vias 0 -> 1
- net Net-(D34-Pad1): track 0.00 -> 138.8 mm, vias 0 -> 1
- net SPI_MOSI1: track 135.8 -> 0.00 mm, vias 3 -> 0
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- removed copper zone on In1.Cu, net GND
- removed copper zone on In2.Cu, net GND
Other:
- board size 299.9 x 215.6 mm -> 300 x 250 mm
- copper layers 4 -> 2
- board text added: "+12V GND Spannungsversorgung"
- board text added: "3,3V GND D 1Wire"
- board text added: "3,3V GND RX TX Serial 1"
- board text added: "3,3V GND RX TX Serial 2"
- board text added: "3,3V GND RX TX Serial 3"
- board text added: "3,3V GND RX TX Serial 4"
- board text added: "3,3V GND RX TX Serial 5"
- board text added: "3,3V GND RX TX Serial 6"
- board text added: "3,3V GND SDA SCL I2C"
- board text added: "Bildschirm AN"
- board text added: "Controller"
- board text added: "DIN 0"
- board text added: "DIN 1"
- board text added: "DIN 10"
- board text added: "DIN 11"
- board text added: "DIN 12"
- board text added: "DIN 13"
- board text added: "DIN 14"
- board text added: "DIN 15"
- board text added: "DIN 16"
- board text added: "DIN 17"
- board text added: "DIN 18"
- board text added: "DIN 19"
- board text added: "DIN 2"
- board text added: "DIN 20"
- board text added: "DIN 21"
- board text added: "DIN 22"
- board text added: "DIN 23"
- board text added: "DIN 24"
- board text added: "DIN 25"
- board text added: "DIN 26"
- board text added: "DIN 27"
- board text added: "DIN 28"
- board text added: "DIN 29"
- board text added: "DIN 3"
- board text added: "DIN 30"
- board text added: "DIN 31"
- board text added: "DIN 4"
- board text added: "DIN 5"
- board text added: "DIN 6"
- board text added: "DIN 7"
- board text added: "DIN 8"
- board text added: "DIN 9"
- board text added: "EA-Platine V0.1"
- board text added: "NC COM NO Relais 1"
- board text added: "NC COM NO Relais 2"
- board text added: "NC COM NO Relais 3"
- board text added: "NC COM NO Relais 4"
- board text added: "NC COM NO Relais 5"
- board text added: "NC COM NO Relais 6"
- board text added: "NC COM NO Relais 7"
- board text added: "NC COM NO Relais 8"
- board text added: "PULLUPs"
- board text removed: "+3.3V"
- board text removed: "+5V"
- board text removed: "12V"
- board text removed: "3,3V"
- board text removed: "3,3V Bypass"
- board text removed: "5V"
- board text removed: "CAN 1"
- board text removed: "CAN 2"
- board text removed: "CAN1"
- board text removed: "CAN2"
- board text removed: "D +3.3V GND"
- board text removed: "DIN_0"
- board text removed: "DIN_1"
- board text removed: "DIN_10"
- board text removed: "DIN_11"
- board text removed: "DIN_12"
- board text removed: "DIN_13"
- board text removed: "DIN_14"
- board text removed: "DIN_15"
- board text removed: "DIN_17"
- board text removed: "DIN_18"
- board text removed: "DIN_19"
- board text removed: "DIN_2"
- board text removed: "DIN_20"
- board text removed: "DIN_21"
- board text removed: "DIN_22"
- board text removed: "DIN_23"
- board text removed: "DIN_24"
- board text removed: "DIN_25"
- board text removed: "DIN_26"
- board text removed: "DIN_27"
- board text removed: "DIN_28"
- board text removed: "DIN_29"
- board text removed: "DIN_3"
- board text removed: "DIN_30"
- board text removed: "DIN_31"
- board text removed: "DIN_32"
- board text removed: "DIN_4"
- board text removed: "DIN_5"
- board text removed: "DIN_6"
- board text removed: "DIN_7"
- board text removed: "DIN_8"
- board text removed: "DIN_9"
- board text removed: "E/A-Platine V2"
- board text removed: "GND"
- board text removed: "LoRa"
- board text removed: "MCP23017"
- board text removed: "Pullup´s"
- board text removed: "RX TX +12V +5V +3.3V GND"
- board text removed: "R_Network08"
- board text removed: "SPI"
- board text removed: "Serial 1"
- board text removed: "Serial 2"
- board text removed: "Serial 3"
- board text removed: "Serial 4"
- board text removed: "Serial 5"
- board text removed: "Serial 6"
- board text removed: "Serial 7"
- board text removed: "Serial 8"
- board text removed: "ULN2803A"
