File: Platine.kicad_sch (KiCad schematic)
At the start: 190 parts, among them J1 GND +12V, J10 RJ45_LED_Shielded, J11 Serial 5, J12 Serial 6, J13 Serial 7, J14 Serial 8, J15 CAN 1, J16 Conn_01x02, J17 Conn_01x02, J18 Conn_01x02, J19 Conn_01x02, J2 Conn_01x09, J20 Conn_01x02, J21 Conn_01x02, J22 Conn_01x02, J23 Conn_01x02, J24 Conn_01x02, J25 Conn_01x02, J26 Conn_01x02, J27 Conn_01x02, J28 Conn_01x02, J29 Conn_01x02, J3 Display128x64_I2C, J30 Conn_01x02, J31 Conn_01x02, J32 +12V, J33 GND, J34 Conn_01x02, J35 Conn_01x02, J36 Conn_01x02, J37 Conn_01x02, J38 Conn_01x02, J39 Conn_01x02, J4 +5V, J40 Conn_01x02, J41 Conn_01x02, J42 Conn_01x02, J43 Conn_01x02, J44 Conn_01x02, J45 Conn_01x02, J46 Conn_01x02, J47 Conn_01x02, J48 Conn_01x02, J49 Conn_01x02, J5 Serial 2, J50 Conn_01x02, J51 Conn_01x02, J52 Conn_01x02, J53 Conn_01x02, J54 Conn_01x02, J55 Conn_01x02, J56 Conn_01x02, J57 Conn_01x02, J58 +12V, J59 GND, J6 Serial 3, J60 Conn_01x02, J61 Conn_01x02, J62 Conn_01x02, J63 Conn_01x02, J64 Conn_01x02, J65 Conn_01x02, J66 Conn_01x02, J67 Conn_01x02, J68 Relais 1, J69 Relais 2, J7 Conn_01x24_Female, J70 Relais 3, J71 Relais 4, J72 Relais 5, J73 Relais 6, J74 Relais 7, J75 Relais 8, J76 +3.3V, J77 GND, J78 +3.3V, J79 GND, J8 Conn_01x24_Female, J80 +5V, J81 GND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

Commit message: ..
Parts:
- removed C1: 100nF, Capacitor_SMD:C_0805_2012Metric_Pad1.18x1.45mm_HandSolder, symbol Device:C
- removed C10, C12: C_Polarized, Capacitor_THT:CP_Radial_D6.3mm_P2.50mm, symbol Device:C_Polarized
- removed C4: C, Capacitor_THT:C_Disc_D3.0mm_W1.6mm_P2.50mm, symbol Device:C
- removed D42, D43, D44: LED, LED_THT:LED_D3.0mm, symbol Device:LED
- removed F1: 12V, Fuse:Fuseholder_TR5_Littelfuse_No560_No460, symbol Device:Fuse
- removed F2: 5V, Fuse:Fuseholder_TR5_Littelfuse_No560_No460, symbol Device:Fuse
- removed F3: 3.3V, Fuse:Fuseholder_TR5_Littelfuse_No560_No460, symbol Device:Fuse
- removed J1: GND +12V, AA_EigeneBauteile:TerminalBlock_MetzConnect_Type166_1x02_P3.50mm_Horizontal, symbol Connector_Generic:Conn_01x02
- removed J10: RJ45_LED_Shielded, Connector_RJ:RJ45_Cetus_J1B1211CCD_Horizontal, symbol Connector:RJ45_LED_Shielded
- removed J11: Serial 5, TerminalBlock_MetzConnect:TerminalBlock_MetzConnect_Type059_RT06306HBWC_1x06_P3.50mm_Horizontal, symbol Connector_Generic:Conn_01x06
- removed J12: Serial 6, TerminalBlock_MetzConnect:TerminalBlock_MetzConnect_Type059_RT06306HBWC_1x06_P3.50mm_Horizontal, symbol Connector_Generic:Conn_01x06
- removed J13: Serial 7, TerminalBlock_MetzConnect:TerminalBlock_MetzConnect_Type059_RT06306HBWC_1x06_P3.50mm_Horizontal, symbol Connector_Generic:Conn_01x06
- removed J14: Serial 8, TerminalBlock_MetzConnect:TerminalBlock_MetzConnect_Type059_RT06306HBWC_1x06_P3.50mm_Horizontal, symbol Connector_Generic:Conn_01x06
- removed J15: CAN 1, TerminalBlock_MetzConnect:TerminalBlock_MetzConnect_Type059_RT06306HBWC_1x06_P3.50mm_Horizontal, symbol Connector_Generic:Conn_01x06
- removed J16, J17, J18, J19, J20, J21, J22, J23, J24, J25, J26, J27, J28, J29, J30, J31, J34, J35, J36, J37, J38, J39, J40, J41, J42, J43, J44, J45, J46, J47, J48, J49, J50, J51, J52, J53, J54, J55, J56, J57, J60, J61, J62, J63, J64, J65, J66, J67: Conn_01x02, AA_EigeneBauteile:TerminalBlock_MetzConnect_Type166_1x02_P3.50mm_Horizontal, symbol Connector_Generic:Conn_01x02
- removed J2: Conn_01x09, AA_EigeneBauteile:PinSocket_1x9_P2.54mm_Vertical_SMD, symbol Connector_Generic:Conn_01x09
- removed J3: Display128x64_I2C, AA_EigeneBauteile:Display128x64_I2C_SMD, symbol Connector_Generic:Conn_01x04
- removed J32, J58, J94: +12V, AA_EigeneBauteile:TerminalBlock_MetzConnect_Type166_1x03_P3.50mm_Horizontal, symbol Connector_Generic:Conn_01x03
- removed J33, J59, J77, J93, J95: GND, AA_EigeneBauteile:TerminalBlock_MetzConnect_Type166_1x03_P3.50mm_Horizontal, symbol Connector_Generic:Conn_01x03
- removed J4: +5V, AA_EigeneBauteile:TerminalBlock_MetzConnect_Type166_1x03_P3.50mm_Horizontal, symbol Connector_Generic:Conn_01x03
- removed J5: Serial 2, TerminalBlock_MetzConnect:TerminalBlock_MetzConnect_Type059_RT06306HBWC_1x06_P3.50mm_Horizontal, symbol Connector_Generic:Conn_01x06
- removed J6: Serial 3, TerminalBlock_MetzConnect:TerminalBlock_MetzConnect_Type059_RT06306HBWC_1x06_P3.50mm_Horizontal, symbol Connector_Generic:Conn_01x06
- removed J68: Relais 1, AA_EigeneBauteile:TerminalBlock_MetzConnect_Type166_1x03_P3.50mm_Horizontal, symbol Connector_Generic:Conn_01x03
- removed J69: Relais 2, AA_EigeneBauteile:TerminalBlock_MetzConnect_Type166_1x03_P3.50mm_Horizontal, symbol Connector_Generic:Conn_01x03
- removed J70: Relais 3, AA_EigeneBauteile:TerminalBlock_MetzConnect_Type166_1x03_P3.50mm_Horizontal, symbol Connector_Generic:Conn_01x03
- removed J71: Relais 4, AA_EigeneBauteile:TerminalBlock_MetzConnect_Type166_1x03_P3.50mm_Horizontal, symbol Connector_Generic:Conn_01x03
- removed J72: Relais 5, AA_EigeneBauteile:TerminalBlock_MetzConnect_Type166_1x03_P3.50mm_Horizontal, symbol Connector_Generic:Conn_01x03
- removed J73: Relais 6, AA_EigeneBauteile:TerminalBlock_MetzConnect_Type166_1x03_P3.50mm_Horizontal, symbol Connector_Generic:Conn_01x03
- removed J74: Relais 7, AA_EigeneBauteile:TerminalBlock_MetzConnect_Type166_1x03_P3.50mm_Horizontal, symbol Connector_Generic:Conn_01x03
- removed J75: Relais 8, AA_EigeneBauteile:TerminalBlock_MetzConnect_Type166_1x03_P3.50mm_Horizontal, symbol Connector_Generic:Conn_01x03
- removed J76: +3.3V, AA_EigeneBauteile:TerminalBlock_MetzConnect_Type166_1x03_P3.50mm_Horizontal, symbol Connector_Generic:Conn_01x03
- removed J78: +3.3V, AA_EigeneBauteile:TerminalBlock_MetzConnect_Type166x1x05_P3.50mm_Horizontal, symbol Connector_Generic:Conn_01x05
- removed J79, J81, J90: GND, AA_EigeneBauteile:TerminalBlock_MetzConnect_Type166x1x05_P3.50mm_Horizontal, symbol Connector_Generic:Conn_01x05
- removed J80: +5V, AA_EigeneBauteile:TerminalBlock_MetzConnect_Type166x1x05_P3.50mm_Horizontal, symbol Connector_Generic:Conn_01x05
- removed J82: CAN-Module1, AA_EigeneBauteile:CAN_Pinsocket_SMD, symbol Connector_Generic:Conn_01x06
- removed J83: CAN-Module2, AA_EigeneBauteile:CAN_Pinsocket_SMD, symbol Connector_Generic:Conn_01x06
- removed J84: CAN 2, TerminalBlock_MetzConnect:TerminalBlock_MetzConnect_Type059_RT06306HBWC_1x06_P3.50mm_Horizontal, symbol Connector_Generic:Conn_01x06
- removed J85: 1Wire, AA_EigeneBauteile:TerminalBlock_MetzConnect_Type166_1x03_P3.50mm_Horizontal, symbol Connector_Generic:Conn_01x03
- removed J86: SPI, AA_EigeneBauteile:SPI_Pinsocket_SMD, symbol Connector_Generic:Conn_01x09
- removed J87, J88, J97: Conn_01x02, Connector_PinHeader_2.54mm:PinHeader_1x02_P2.54mm_Vertical, symbol Connector_Generic:Conn_01x02
- removed J89: +12V, AA_EigeneBauteile:TerminalBlock_MetzConnect_Type166x1x05_P3.50mm_Horizontal, symbol Connector_Generic:Conn_01x05
- removed J9: Serial 4, TerminalBlock_MetzConnect:TerminalBlock_MetzConnect_Type059_RT06306HBWC_1x06_P3.50mm_Horizontal, symbol Connector_Generic:Conn_01x06
- removed J91: Serial 1, TerminalBlock_MetzConnect:TerminalBlock_MetzConnect_Type059_RT06306HBWC_1x06_P3.50mm_Horizontal, symbol Connector_Generic:Conn_01x06
- removed J92: Pullups´s, AA_EigeneBauteile:DIP-6_W7.62mm_SMD, symbol Connector_Generic:Conn_02x03_Counter_Clockwise
- removed J96: LoRa, AA_EigeneBauteile:LoRa_Pinsocket_SMD, symbol Connector_Generic:Conn_01x09
- removed R10: 68 Ohm, Resistor_SMD:R_0603_1608Metric_Pad0.98x0.95mm_HandSolder, symbol Device:R
- removed R11: 220 Ohm, Resistor_SMD:R_0603_1608Metric_Pad0.98x0.95mm_HandSolder, symbol Device:R
- removed R4, R7: Endwiderst. CAN 120 Ohm, Resistor_SMD:R_0603_1608Metric_Pad0.98x0.95mm_HandSolder, symbol Device:R
- removed R8: PULLUP, Resistor_SMD:R_0805_2012Metric_Pad1.20x1.40mm_HandSolder, symbol Device:R_Small
- removed R9: 560 Ohm, Resistor_SMD:R_0603_1608Metric_Pad0.98x0.95mm_HandSolder, symbol Device:R
- removed U1: OKI-78SR-3.3_1.5-W36-C, Converter_DCDC:Converter_DCDC_Murata_OKI-78SR_Vertical, symbol Converter_DCDC:OKI-78SR-5_1.5-W36-C
- removed U4: MCP23S17_SP, AA_EigeneBauteile:DIP-28_W7.62mm_SMD, symbol Interface_Expansion:MCP23017_SP
- added J1: Spannungsversorgung +12V DC, TerminalBlock_MetzConnect:TerminalBlock_MetzConnect_Type011_RT05504HBWC_1x04_P5.00mm_Horizontal, symbol Connector:Conn_01x04_Male
- added J10: Serial 3, TerminalBlock_MetzConnect:TerminalBlock_MetzConnect_Type011_RT05504HBWC_1x04_P5.00mm_Horizontal, symbol Connector:Conn_01x04_Male
- added J11: Serial 4, TerminalBlock_MetzConnect:TerminalBlock_MetzConnect_Type011_RT05504HBWC_1x04_P5.00mm_Horizontal, symbol Connector:Conn_01x04_Male
- added J12: Serial 5, TerminalBlock_MetzConnect:TerminalBlock_MetzConnect_Type011_RT05504HBWC_1x04_P5.00mm_Horizontal, symbol Connector:Conn_01x04_Male
- added J13: Serial 6, TerminalBlock_MetzConnect:TerminalBlock_MetzConnect_Type011_RT05504HBWC_1x04_P5.00mm_Horizontal, symbol Connector:Conn_01x04_Male
- added J14: I2C, TerminalBlock_MetzConnect:TerminalBlock_MetzConnect_Type011_RT05504HBWC_1x04_P5.00mm_Horizontal, symbol Connector:Conn_01x04_Male
- added J15: 1Wire, TerminalBlock_MetzConnect:TerminalBlock_MetzConnect_Type011_RT05504HBWC_1x04_P5.00mm_Horizontal, symbol Connector:Conn_01x04_Male
- added J16, J41: Digitale Eingänge, TerminalBlock_MetzConnect:TerminalBlock_MetzConnect_Type011_RT05502HBWC_1x02_P5.00mm_Horizontal, symbol Connector:Conn_01x02_Male
- added J17, J18, J19, J20, J21, J22, J23, J24, J25, J26, J27, J28, J29, J30, J31, J32, J33, J34, J35, J36, J37, J38, J39, J42, J43, J44, J45, J46, J47, J48, J49, J50, J51, J52, J53, J54, J55, J56, J57, J58, J59, J60, J61, J62, J63, J64: Conn_01x02_Male, TerminalBlock_MetzConnect:TerminalBlock_MetzConnect_Type011_RT05502HBWC_1x02_P5.00mm_Horizontal, symbol Connector:Conn_01x02_Male
- added J2: Spannungsversorgung GND, TerminalBlock_MetzConnect:TerminalBlock_MetzConnect_Type011_RT05504HBWC_1x04_P5.00mm_Horizontal, symbol Connector:Conn_01x04_Male
- added J3, J4: Conn_01x03_Female, Connector_PinSocket_2.54mm:PinSocket_1x03_P2.54mm_Vertical, symbol Connector:Conn_01x03_Female
- added J40, J65: Digitale Ausgänge, TerminalBlock_MetzConnect:TerminalBlock_MetzConnect_Type011_RT05502HBWC_1x02_P5.00mm_Horizontal, symbol Connector:Conn_01x02_Male
- added J5: Serial 1 - NFC-Reader 1, TerminalBlock_MetzConnect:TerminalBlock_MetzConnect_Type011_RT05504HBWC_1x04_P5.00mm_Horizontal, symbol Connector:Conn_01x04_Male
- added J6: I2C-Display, AA_EigeneBauteile:Display128x64_I2C, symbol Connector:Conn_01x04_Male
- added J66: Relais 1, TerminalBlock_MetzConnect:TerminalBlock_MetzConnect_Type055_RT01503HDWU_1x03_P5.00mm_Horizontal, symbol Connector:Conn_01x03_Male
- added J67: Relais 2, TerminalBlock_MetzConnect:TerminalBlock_MetzConnect_Type055_RT01503HDWU_1x03_P5.00mm_Horizontal, symbol Connector:Conn_01x03_Male
- added J68: Relais 3, TerminalBlock_MetzConnect:TerminalBlock_MetzConnect_Type055_RT01503HDWU_1x03_P5.00mm_Horizontal, symbol Connector:Conn_01x03_Male
- added J69: Relais 4, TerminalBlock_MetzConnect:TerminalBlock_MetzConnect_Type055_RT01503HDWU_1x03_P5.00mm_Horizontal, symbol Connector:Conn_01x03_Male
- added J7: Serial 2 - NFC-Reader 2, TerminalBlock_MetzConnect:TerminalBlock_MetzConnect_Type011_RT05504HBWC_1x04_P5.00mm_Horizontal, symbol Connector:Conn_01x04_Male
- added J70: Relais 5, TerminalBlock_MetzConnect:TerminalBlock_MetzConnect_Type055_RT01503HDWU_1x03_P5.00mm_Horizontal, symbol Connector:Conn_01x03_Male
- added J71: Relais 6, TerminalBlock_MetzConnect:TerminalBlock_MetzConnect_Type055_RT01503HDWU_1x03_P5.00mm_Horizontal, symbol Connector:Conn_01x03_Male
- added J72: Relais 7, TerminalBlock_MetzConnect:TerminalBlock_MetzConnect_Type055_RT01503HDWU_1x03_P5.00mm_Horizontal, symbol Connector:Conn_01x03_Male
- added J73: Relais 8, TerminalBlock_MetzConnect:TerminalBlock_MetzConnect_Type055_RT01503HDWU_1x03_P5.00mm_Horizontal, symbol Connector:Conn_01x03_Male
- C1: renamed from C11; footprint Capacitor_THT:CP_Radial_D6.3mm_P2.50mm -> Capacitor_SMD:CP_Elec_4x5.4
- J8: renamed from J7; footprint AA_EigeneBauteile:PinSocket_1x24_P2.54mm_Vertical_SMD -> Connector_PinSocket_2.54mm:PinSocket_1x24_P2.54mm_Vertical
- J9: renamed from J8; footprint AA_EigeneBauteile:PinSocket_1x24_P2.54mm_Vertical_SMD -> Connector_PinSocket_2.54mm:PinSocket_1x24_P2.54mm_Vertical
- RN1, RN2, RN3, RN4, RN5: footprint AA_EigeneBauteile:PinSocket_1x9_P2.54mm_Vertical_SMD -> Resistor_THT:R_Array_SIP9
- U2: renamed from U3; footprint AA_EigeneBauteile:Teensy41_without_some_pins_SMD -> teensy:Teensy41
- renumbered C3 to C2, C5 to C3, C6 to C4, C7 to C5, C8 to C6, R3 to R1, R4 to R2, R5 to R3, R6 to R4, U2 to U1, U12 to U10, U13 to U11, U5 to U3, U6 to U4, U7 to U5, U8 to U6, U9 to U7, U10 to U8, U11 to U9
Connections:
- net +12V.1 is gone; now on net +12V: K1.A2, K2.A2, K3.A2, K4.A2, K5.A2, K6.A2, K7.A2, K8.A2, RN1.1 (common), RN2.1 (common), RN3.1 (common), RN4.1 (common), RN5.1 (common), U10.10 (COM), U11.10 (COM), U3.10 (COM), U6.10 (COM), U7.10 (COM)
- net +3.3V is gone; now on net +3V3: C3.1, C4.1, C5.1, C6.1, R1.1, R2.1, R3.1, R4.1, U4.16 (A1), U4.9 (VDD), U5.9 (VDD), U8.15 (A0), U8.16 (A1), U8.9 (VDD), U9.15 (A0), U9.9 (VDD)
- net LoRa_IRQ is gone; now on net Taster: J9.16 (Pin_16), U2.33 (41_A17)
- net LoRa_Reset is gone; now on net Relais 8: J9.17 (Pin_17), U2.32 (40_A16)
- net RX8 is gone; now on net Relais 2: J9.23 (Pin_23), U2.26 (34_RX8)
- net Relais1 is gone; now on net Relais 1: J9.24 (Pin_24), U2.25 (33_MCLK2)
- net SPI_CS1 is gone; now on net Relais 6: J9.19 (Pin_19), U2.30 (38_CS1_IN1)
- net SPI_MISO1 is gone; now on net Relais 7: J9.18 (Pin_18), U2.31 (39_MISO1_OUT1A)
- net SPI_MOSI is gone; now on net 1Wire: J8.13 (Pin_13), U2.13 (11_MOSI_CTX1)
- net SPI_SCK is gone; now on net Relais 5: J9.20 (Pin_20), U2.29 (37_CS)
- net TX8 is gone; now on net Relais 3: J9.22 (Pin_22), U2.27 (35_TX8)
- net +12V: now also J1.1 (Pin_1), J1.2 (Pin_2), J1.3 (Pin_3), J1.4 (Pin_4), J32.1 (Pin_1), J32.2 (Pin_2), J57.1 (Pin_1), J57.2 (Pin_2)
- net +5V: now also C1.1, U1.3 (OUT)
- net 1Wire: now also J15.3 (Pin_3), J4.1 (Pin_1); no longer J8.11 (Pin_11), U2.11 (9_OUT1C)
- net GND: now also J10.2 (Pin_2), J11.2 (Pin_2), J12.2 (Pin_2), J13.2 (Pin_2), J14.2 (Pin_2), J15.2 (Pin_2), J16.2 (Pin_2), J17.2 (Pin_2), J18.2 (Pin_2), J19.2 (Pin_2), J2.1 (Pin_1), J2.2 (Pin_2), J2.3 (Pin_3), J2.4 (Pin_4), J20.2 (Pin_2), J21.2 (Pin_2), J22.2 (Pin_2), J23.2 (Pin_2), J24.2 (Pin_2), J25.2 (Pin_2), J26.2 (Pin_2), J27.2 (Pin_2), J28.2 (Pin_2), J29.2 (Pin_2), J30.2 (Pin_2), J31.2 (Pin_2), J41.2 (Pin_2), J42.2 (Pin_2), J43.2 (Pin_2), J44.2 (Pin_2), J45.2 (Pin_2), J46.2 (Pin_2), J47.2 (Pin_2), J48.2 (Pin_2), J49.2 (Pin_2), J5.2 (Pin_2), J50.2 (Pin_2), J51.2 (Pin_2), J52.2 (Pin_2), J53.2 (Pin_2), J54.2 (Pin_2), J55.2 (Pin_2), J56.2 (Pin_2), J6.2 (Pin_2), J7.2 (Pin_2)
- net RX1: now also J5.3 (Pin_3)
- net RX2: now also J7.3 (Pin_3)
- net RX3: now also J10.3 (Pin_3)
- net RX4: now also J11.3 (Pin_3)
- net RX5: now also J12.3 (Pin_3)
- net RX6: now also J13.3 (Pin_3)
- net SCL: now also J14.4 (Pin_4), J4.3 (Pin_3), J6.3 (Pin_3)
- net SDA: now also J14.3 (Pin_3), J4.2 (Pin_2), J6.4 (Pin_4)
- net TX1: now also J5.4 (Pin_4)
- net TX2: now also J7.4 (Pin_4)
- net TX3: now also J10.4 (Pin_4)
- net TX4: now also J11.4 (Pin_4)
- net TX5: now also J12.4 (Pin_4)
- net TX6: now also J13.4 (Pin_4)
- net Taster: no longer J8.4 (Pin_4), U2.4 (2_OUT2)
- net at U5.1 (GPB0): now also J16.1 (Pin_1)
- net at U5.2 (GPB1): now also J17.1 (Pin_1)
- net at U5.21 (GPA0): now also J24.1 (Pin_1)
- net at U5.22 (GPA1): now also J25.1 (Pin_1)
- net at U5.23 (GPA2): now also J26.1 (Pin_1)
- net at U5.24 (GPA3): now also J27.1 (Pin_1)
- net at U5.25 (GPA4): now also J28.1 (Pin_1)
- net at U5.26 (GPA5): now also J29.1 (Pin_1)
- net at U5.27 (GPA6): now also J30.1 (Pin_1)
- net at U5.28 (GPA7): now also J31.1 (Pin_1)
- net at U5.3 (GPB2): now also J18.1 (Pin_1)
- net at U5.4 (GPB3): now also J19.1 (Pin_1)
- net at U5.5 (GPB4): now also J20.1 (Pin_1)
- net at U5.6 (GPB5): now also J21.1 (Pin_1)
- net at U5.7 (GPB6): now also J22.1 (Pin_1)
- net at U5.8 (GPB7): now also J23.1 (Pin_1)
- net at D8.1 (K), U3.11 (O8): now also J36.1 (Pin_1)
- net at D7.1 (K), U3.12 (O7): now also J36.2 (Pin_2)
- net at D6.1 (K), U3.13 (O6): now also J35.1 (Pin_1)
- net at D5.1 (K), U3.14 (O5): now also J35.2 (Pin_2)
- net at D4.1 (K), U3.15 (O4): now also J34.1 (Pin_1)
- net at D3.1 (K), U3.16 (O3): now also J34.2 (Pin_2)
- net at D2.1 (K), U3.17 (O2): now also J33.1 (Pin_1)
- net at D1.1 (K), U3.18 (O1): now also J33.2 (Pin_2)
- net at D16.1 (K), U6.11 (O8): now also J40.1 (Pin_1)
- net at D15.1 (K), U6.12 (O7): now also J40.2 (Pin_2)
- net at D14.1 (K), U6.13 (O6): now also J39.1 (Pin_1)
- net at D13.1 (K), U6.14 (O5): now also J39.2 (Pin_2)
- net at D12.1 (K), U6.15 (O4): now also J38.1 (Pin_1)
- net at D11.1 (K), U6.16 (O3): now also J38.2 (Pin_2)
- net at D10.1 (K), U6.17 (O2): now also J37.1 (Pin_1)
- net at D9.1 (K), U6.18 (O1): now also J37.2 (Pin_2)
- net at U9.1 (GPB0): now also J41.1 (Pin_1)
- net at U9.2 (GPB1): now also J42.1 (Pin_1)
- net at U9.21 (GPA0): now also J49.1 (Pin_1)
- net at U9.22 (GPA1): now also J50.1 (Pin_1)
- net at U9.23 (GPA2): now also J51.1 (Pin_1)
- net at U9.24 (GPA3): now also J52.1 (Pin_1)
- net at U9.25 (GPA4): now also J53.1 (Pin_1)
- net at U9.26 (GPA5): now also J54.1 (Pin_1)
- net at U9.27 (GPA6): now also J55.1 (Pin_1)
- net at U9.28 (GPA7): now also J56.1 (Pin_1)
- net at U9.3 (GPB2): now also J43.1 (Pin_1)
- net at U9.4 (GPB3): now also J44.1 (Pin_1)
- net at U9.5 (GPB4): now also J45.1 (Pin_1)
- net at U9.6 (GPB5): now also J46.1 (Pin_1)
- net at U9.7 (GPB6): now also J47.1 (Pin_1)
- net at U9.8 (GPB7): now also J48.1 (Pin_1)
- net at K8.11: now also J73.2 (Pin_2)
- net at K8.12: now also J73.3 (Pin_3)
- net at K8.14: now also J73.1 (Pin_1)
- net at D40.1 (K), K8.A1: now also U11.11 (O8); no longer U11.18 (O1)
- net at D38.1 (K), K6.A1: now also U11.13 (O6); no longer U11.16 (O3)
- net at D31.1 (K), U10.12 (O7): now also J65.2 (Pin_2)
- net at D32.1 (K), U10.11 (O8): now also J65.1 (Pin_1)
- net Relais 4: now reaches J9.21 (Pin_21), U2.28 (36_CS)
- net Relais 4: now also U11.4 (I4)
- net +3V3: now reaches J9.3 (Pin_3), U2.46 (3V3)
- net +3V3: now also J10.1 (Pin_1), J11.1 (Pin_1), J12.1 (Pin_1), J13.1 (Pin_1), J14.1 (Pin_1), J15.1 (Pin_1), J3.1 (Pin_1), J3.2 (Pin_2), J3.3 (Pin_3), J5.1 (Pin_1), J6.1 (Pin_1), J7.1 (Pin_1)
- net at D23.1 (K), U7.12 (O7): now also J61.2 (Pin_2)
- net at D24.1 (K), U7.11 (O8): now also J61.1 (Pin_1)
- net at D29.1 (K), U10.14 (O5): now also J64.2 (Pin_2)
- net at D30.1 (K), U10.13 (O6): now also J64.1 (Pin_1)
- net at D28.1 (K), U10.15 (O4): now also J63.1 (Pin_1)
- net at D27.1 (K), U10.16 (O3): now also J63.2 (Pin_2)
- net at D26.1 (K), U10.17 (O2): now also J62.1 (Pin_1)
- net at D25.1 (K), U10.18 (O1): now also J62.2 (Pin_2)
- net at D22.1 (K), U7.13 (O6): now also J60.1 (Pin_1)
- net at K3.14: now also J68.1 (Pin_1)
- net at K3.11: now also J68.2 (Pin_2)
- net at K3.12: now also J68.3 (Pin_3)
- net at K5.14: now also J70.1 (Pin_1)
- net at K5.11: now also J70.2 (Pin_2)
- net at K5.12: now also J70.3 (Pin_3)
- net at K2.11: now also J67.2 (Pin_2)
- net at K2.12: now also J67.3 (Pin_3)
- net at K2.14: now also J67.1 (Pin_1)
- net at D34.1 (K), K2.A1: now also U11.17 (O2); no longer U11.12 (O7)
- net Relais 1: now reaches U11.1 (I1)
- net at D33.1 (K), K1.A1: now also U11.18 (O1); no longer U11.11 (O8)
- net at D35.1 (K), K3.A1: now also U11.16 (O3); no longer U11.13 (O6)
- net at D36.1 (K), K4.A1: now also U11.15 (O4); no longer U11.14 (O5)
- net at D37.1 (K), K5.A1: now also U11.14 (O5); no longer U11.15 (O4)
- net at D39.1 (K), K7.A1: now also U11.12 (O7); no longer U11.17 (O2)
- net Relais 2: now reaches U11.2 (I2)
- net Relais 3: now reaches U11.3 (I3)
- net Relais 5: now reaches U11.5 (I5)
- net Relais 6: now reaches U11.6 (I6)
- net Relais 7: now reaches U11.7 (I7)
- net Relais 8: now reaches U11.8 (I8)
- net at K4.14: now also J69.1 (Pin_1)
- net at K4.11: now also J69.2 (Pin_2)
- net at K4.12: now also J69.3 (Pin_3)
- net at K6.14: now also J71.1 (Pin_1)
- net at K6.11: now also J71.2 (Pin_2)
- net at K6.12: now also J71.3 (Pin_3)
- net at D18.1 (K), U7.17 (O2): now also J58.1 (Pin_1)
- net at D19.1 (K), U7.16 (O3): now also J59.2 (Pin_2)
- net at D20.1 (K), U7.15 (O4): now also J59.1 (Pin_1)
- net at D21.1 (K), U7.14 (O5): now also J60.2 (Pin_2)
- net at D17.1 (K), U7.18 (O1): now also J58.2 (Pin_2)
- net at K7.14: now also J72.1 (Pin_1)
- net at K7.11: now also J72.2 (Pin_2)
- net at K7.12: now also J72.3 (Pin_3)
- net at K1.14: now also J66.1 (Pin_1)
- net at K1.11: now also J66.2 (Pin_2)
- net at K1.12: now also J66.3 (Pin_3)
- net CAN1_RX: no longer names the net of J9.4 (Pin_4), U2.45 (23_A9_CRX1_MCLK1)
- net CAN1_TX: no longer names the net of J9.5 (Pin_5), U2.44 (22_A8_CTX1)
- net CAN2_RX: no longer names the net of J8.22 (Pin_22), U2.22 (30_CRX3)
- net CAN2_TX: no longer names the net of J8.23 (Pin_23), U2.23 (31_CTX3)
- net LED_LOOP: no longer names the net of J8.24 (Pin_24), U2.24 (32_OUT1B)
- net MCP0_INTA: no longer names the net of J8.6 (Pin_6), U2.6 (4_BCLK2)
- net MCP0_INTA: no longer U5.20 (INTA)
- net MCP0_INTB: no longer names the net of J8.5 (Pin_5), U2.5 (3_LRCLK2)
- net MCP0_INTB: no longer U5.19 (INTB)
- net MCP1_INTA: no longer names the net of J8.7 (Pin_7), U2.7 (5_IN2)
- net MCP1_INTA: no longer U9.20 (INTA)
- net MCP1_INTB: no longer names the net of J8.8 (Pin_8), U2.8 (6_OUT1D)
- net MCP1_INTB: no longer U9.19 (INTB)
- net RX7: no longer names the net of J8.20 (Pin_20), U2.20 (28_RX7)
- net SPI_CS: no longer names the net of J8.12 (Pin_12), U2.12 (10_CS_MQSR)
- net SPI_MISO: no longer names the net of J8.14 (Pin_14), U2.14 (12_MISO_MQSL)
- net SPI_MOSI1: no longer names the net of J8.18 (Pin_18), U2.18 (26_A12_MOSI1)
- net SPI_SCK1: no longer names the net of J8.19 (Pin_19), U2.19 (27_A13_SCK1)
- net SPI_SCK_umgelötet: no longer names the net of J9.14 (Pin_14), U2.35 (13_SCK_LED)
- net TX7: no longer names the net of J8.21 (Pin_21), U2.21 (29_TX7)
- new net: J8.11 (Pin_11), U2.11 (9_OUT1C)
- new net: J8.4 (Pin_4), U2.4 (2_OUT2)
- no-connect marks 6 -> 8
Other:
- note removed: "000"
- note removed: "010"
- note removed: "100"
- note removed: "110"
- note removed: "111"
- moved on the sheet: C1, C2, C3, C4, C5, C6, D1, D10, D11, D12, D13, D14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
