File: Platine.kicad_sch (KiCad schematic)
At the start: 190 parts, among them J1 GND +12V, J10 RJ45_LED_Shielded, J11 Serial 5, J12 Serial 6, J13 Serial 7, J14 Serial 8, J15 CAN 1, J16 Conn_01x02, J17 Conn_01x02, J18 Conn_01x02, J19 Conn_01x02, J2 Conn_01x09, J20 Conn_01x02, J21 Conn_01x02, J22 Conn_01x02, J23 Conn_01x02, J24 Conn_01x02, J25 Conn_01x02, J26 Conn_01x02, J27 Conn_01x02, J28 Conn_01x02, J29 Conn_01x02, J3 Display128x64_I2C, J30 Conn_01x02, J31 Conn_01x02, J32 +12V, J33 GND, J34 Conn_01x02, J35 Conn_01x02, J36 Conn_01x02, J37 Conn_01x02, J38 Conn_01x02, J39 Conn_01x02, J4 +5V, J40 Conn_01x02, J41 Conn_01x02, J42 Conn_01x02, J43 Conn_01x02, J44 Conn_01x02, J45 Conn_01x02, J46 Conn_01x02, J47 Conn_01x02, J48 Conn_01x02, J49 Conn_01x02, J5 Serial 2, J50 Conn_01x02, J51 Conn_01x02, J52 Conn_01x02, J53 Conn_01x02, J54 Conn_01x02, J55 Conn_01x02, J56 Conn_01x02, J57 Conn_01x02, J58 +12V, J59 GND, J6 Serial 3, J60 Conn_01x02, J61 Conn_01x02, J62 Conn_01x02, J63 Conn_01x02, J64 Conn_01x02, J65 Conn_01x02, J66 Conn_01x02, J67 Conn_01x02, J68 Relais 1, J69 Relais 2, J7 Conn_01x24_Female, J70 Relais 3, J71 Relais 4, J72 Relais 5, J73 Relais 6, J74 Relais 7, J75 Relais 8, J76 +3.3V, J77 GND, J78 +3.3V, J79 GND, J8 Conn_01x24_Female, J80 +5V, J81 GND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

Commit message: ..
Parts:
- renumbered R4 to R1
